Commit message: minor correction

File: bot_description/urdf/bot.urdf.xacro (robot description, xacro)
@@ -2,5 +2,5 @@
 <robot name="bot" xmlns:xacro="http://www.ros.org/wiki/xacro">
     <xacro:include filename="common_properties.xacro" />
-    <link name="base_footprint" />
+    <!-- <link name="base_footprint" /> -->
     <link name="base_link">
         <visual>
@@ -8,5 +8,5 @@
                 <box size="0.2 0.2 0.1" />
             </geometry>
-            <origin xyz="0 0 0.05" rpy="0 0 0" />
+            <origin xyz="0 0 0" rpy="0 0 0" />
             <material name="blue" />
         </visual>
@@ -15,8 +15,8 @@
                 <box size="0.2 0.2 0.1" />
             </geometry>
-            <origin xyz="0 0 0.05" rpy="0 0 0" />
+            <origin xyz="0 0 0" rpy="0 0 0" />
         </collision>
         <xacro:box_inertia m="2.5" l="0.2" w="0.2" h="0.1"
-            xyz="0 0 0.05" rpy="0 0 0" />
+            xyz="0 0 0" rpy="0 0 0" />
     </link>
     <link name="right_wheel_link">
@@ -69,14 +69,14 @@
     </link>
     <!-- Fixed joint to place base_link at correct height -->
-    <joint name="base_joint" type="fixed">
+    <!-- <joint name="base_joint" type="fixed">
         <parent link="base_footprint"/>
         <child link="base_link"/>
         <origin xyz="0 0 0.05" rpy="0 0 0"/>
-    </joint>
+    </joint> -->
     <!-- Wheel joints with precise positioning -->
     <joint name="base_right_wheel_joint" type="continuous">
         <parent link="base_link"/>
         <child link="right_wheel_link"/>
-        <origin xyz="-0.035 -0.105 0.05" rpy="0 0 0"/>
+        <origin xyz="-0.035 -0.105 0" rpy="0 0 0"/>
         <axis xyz="0 1 0"/>
     </joint>
@@ -84,5 +84,5 @@
         <parent link="base_link"/>
         <child link="left_wheel_link"/>
-        <origin xyz="-0.035 0.105 0.05" rpy="0 0 0"/>
+        <origin xyz="-0.035 0.105 0" rpy="0 0 0"/>
         <axis xyz="0 1 0"/>
     </joint>
@@ -90,5 +90,5 @@
         <parent link="base_link"/>
         <child link="caster_wheel_link"/>
-        <origin xyz="0.071 0 0.01" rpy="0 0 0"/>
+        <origin xyz="0.071 0 -0.05" rpy="0 0 0"/>
         <dynamics damping="0.0" friction="0.01"/>
     </joint>

Commit message: minor correction

File: bot_description/urdf/bot.urdf.xacro (robot description, xacro)
@@ -90,6 +90,6 @@
         <parent link="base_link"/>
         <child link="caster_wheel_link"/>
-        <origin xyz="0.071 0 -0.05" rpy="0 0 0"/>
-        <dynamics damping="0.0" friction="0.01"/>
+        <origin xyz="0.071 0 -0.039" rpy="0 0 0"/>
+        <!-- <dynamics damping="0.0" friction="0.01"/> -->
     </joint>
     <!-- Lidar Link -->
